File: ECAD/iridium-stack.kicad_sch (KiCad schematic)
At the start: 28 parts

Commit message: current monitor
Parts:
- added C?: (no value), symbol Device:C
- added R?: (no value), symbol Device:R
- added TP?: (no value), symbol Connector:TestPoint
- added U?: (no value), symbol Amplifier_Current:INA138
- A1: footprint (none) -> 9602:9602
- C10, C11: value (none) -> 22uF; footprint (none) -> Capacitor_SMD:C_1210_3225Metric
- C12, C13: footprint (none) -> Capacitor_Tantalum_SMD:CP_EIA-7343-43_Kemet-X_Pad2.25x2.55mm_HandSolder
- C7: value (none) -> 2.2uF
- C8: value (none) -> 47nF
- J1: value (none) -> Header; footprint (none) -> Connector_PinHeader_2.54mm:PinHeader_1x11_P2.54mm_Vertical
- L1: footprint (none) -> Inductor_SMD:L_AVX_LMLP07A7
- R1: value (none) -> 26.3K; footprint (none) -> Resistor_SMD:R_1206_3216Metric
- TP1, TP2: footprint (none) -> TestPoint:TestPoint_2Pads_Pitch5.08mm_Drill1.3mm
- TP3: footprint (none) -> TestPoint:TestPoint_Pad_3.0x3.0mm
- U1: value (none) -> MAX17644; footprint (none) -> Package_DFN_QFN:TQFN-16-1EP_3x3mm_P0.5mm_EP1.23x1.23mm_ThermalVias
Connections:
- net +5VP: now also C?.1, R?.2, U?.4 (-), U?.5 (V+); no longer C10.1, C11.1, C12.1, C13.1, L1.2, TP2.2, U1.6 (FB), U1.9 (EXTVCC)
- net GND: now also C?.2, U?.2 (GND)
- new net: C10.1, C11.1, C12.1, C13.1, L1.2, R?.1, TP2.2, U1.6 (FB), U1.9 (EXTVCC), U?.3 (+)
- new net IDRAW: TP?.1, U?.1
